File: hardware/solar/cad/mcu.kicad_sch (KiCad schematic)
At the start: 0 parts

Commit message: Attempt to roll our own charging but stop before I get carried away
This is actually a real pain in the ass, so we're not going to deal with
it yet. My thoughts are that we should focus on getting something out
the door otherwise I'm going to spend a long time designing a NiMH
charger.

Some problem/open questions in this design:
 - Constant current driver uses a lot of power if we want to support
   fast charging. ~3W of the 6W available.
 - Some kind of switching regulator would be more suited to the task I
   think. BQ24401 seems like a suitable part, relatively cheap.
 - Need an accurate (~1mV according to one source I read) voltage
   sensing circuit if we want to do ∆V/dt termination.

Saving this in this branch to inspire future improvements when we can
prove we need them.
Changed lines of the file:
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@@
+    (effects (font (size 1.27 1.27)) (justify left))
+  )
+  (hierarchical_label "GND" (shape passive) (at 96.52 97.79 0)
+    (effects (font (size 1.27 1.27)) (justify left))
+  )
+  (hierarchical_label "VDD" (shape passive) (at 96.52 69.85 0)
     (effects (font (size 1.27 1.27)) (justify left))
   )
   (hierarchical_label "I2C" (shape bidirectional) (at 96.52 95.25 0)
+    (effects (font (size 1.27 1.27)) (justify left))
+  )
+  (hierarchical_label "~{CS}" (shape input) (at 96.52 77.47 0)
     (effects (font (size 1.27 1.27)) (justify left))
   )
@@
     (effects (font (size 1.27 1.27)) (justify left))
   )
+  (hierarchical_label "SCK" (shape input) (at 96.52 72.39 0)
+    (effects (font (size 1.27 1.27)) (justify left))
+  )
   (hierarchical_label "VSENSE_NTC" (shape input) (at 96.52 80.01 0)
     (effects (font (size 1.27 1.27)) (justify left))
   )
+  (hierarchical_label "SDI" (shape input) (at 96.52 74.93 0)
+    (effects (font (size 1.27 1.27)) (justify left))
+  )
